File: ftdi_adapter.brd (EAGLE design)
At the start: 14.5 x 16.3 mm, 4 parts, among them J2 UPDI COMPACT, J3 6PIN SERIAL

Commit message: initial version
Parts:
- added JMP1: PWR, bt:JUMPER-2W-PIN-0.1IN
- moved J2 5.59 mm to (18.3, 8.13)
- moved D1 5.09 mm to (5.59, 10.7), turned to 90 degrees
- moved U$1 1.02 mm to (6.60, 12.7), flipped to the top, turned to 0 degrees
Connections:
- new net DATA: D1.A, J2.3, J3.2
- net GND: now also J3.6; no longer J3.1
- net N$1: now also J3.3; no longer J3.4
- net N$2: now also J3.4, JMP1.2; no longer D1.A, J2.3, J3.5
- net VCC: now also JMP1.1; no longer J3.3
Routing:
- net DATA: track 0.00 -> 17.5 mm
- net N$2: track 13.6 -> 8.91 mm, vias 1 -> 0
- net VCC: track 12.5 -> 8.13 mm
Other:
- board size 14.5 x 16.3 mm -> 20.1 x 16.3 mm
- board text added: "5V>VDD"
Changed lines of the file:
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@@
 <wire x1="0" y1="15.621" x2="0" y2="0.635" width="0" layer="20"/>
 <wire x1="0" y1="0.635" x2="0.635" y2="0" width="0" layer="20" curve="90"/>
-<wire x1="0.635" y1="0" x2="11.938" y2="0" width="0" layer="20"/>
-<wire x1="11.938" y1="0" x2="14.478" y2="2.54" width="0" layer="20"/>
-<wire x1="14.478" y1="2.54" x2="14.478" y2="13.716" width="0" layer="20"/>
-<wire x1="14.478" y1="13.716" x2="11.938" y2="16.256" width="0" layer="20"/>
-<wire x1="11.938" y1="16.256" x2="0.635" y2="16.256" width="0" layer="20"/>
+<wire x1="0.635" y1="0" x2="19.431" y2="0" width="0" layer="20"/>
+<wire x1="19.431" y1="0" x2="20.066" y2="0.635" width="0" layer="20" curve="90"/>
+<wire x1="20.066" y1="0.635" x2="20.066" y2="15.621" width="0" layer="20"/>
+<wire x1="20.066" y1="15.621" x2="19.431" y2="16.256" width="0" layer="20" curve="90"/>
+<wire x1="19.431" y1="16.256" x2="0.635" y2="16.256" width="0" layer="20"/>
 <wire x1="0.635" y1="16.256" x2="0" y2="15.621" width="0" layer="20" curve="90"/>
-<text x="8.636" y="1.016" size="1.016" layer="25" font="vector" ratio="10" align="bottom-center">UPDI
-Adapter</text>
-<text x="7.62" y="0.762" size="0.8128" layer="26" font="vector" ratio="10" rot="MR0" align="bottom-center">cc-by-sa</text>
-<text x="13.716" y="13.716" size="0.8128" layer="25" font="vector" ratio="10" rot="R135">R0.1</text>
-<text x="11.176" y="10.668" size="0.8128" layer="25" font="vector" ratio="10" align="center-right">UPDI</text>
-<text x="11.176" y="5.588" size="0.8128" layer="25" font="vector" ratio="10" align="center-right">VDD</text>
-<text x="11.176" y="8.128" size="0.8128" layer="25" font="vector" ratio="10" align="center-right">GND</text>
-<text x="5.588" y="15.494" size="0.8128" layer="26" font="vector" ratio="10" rot="MR90" align="bottom-right">bot-thoughts.com</text>
+<text x="11.684" y="1.016" size="1.016" layer="25" font="vector" ratio="10" align="bottom-center">UPDI Adapter</text>
+<text x="8.636" y="13.462" size="0.8128" layer="25" font="vector" ratio="10">cc-by-sa</text>
+<text x="19.558" y="1.27" size="0.8128" layer="25" font="vector" ratio="10" rot="R90">R0.1</text>
+<text x="17.018" y="10.922" size="0.8128" layer="25" font="vector" ratio="10" rot="R90" align="bottom-center">UPDI</text>
+<text x="17.018" y="5.588" size="0.8128" layer="25" font="vector" ratio="10" rot="R90" align="bottom-center">VDD</text>
+<text x="17.018" y="8.128" size="0.8128" layer="25" font="vector" ratio="10" rot="R90" align="bottom-center">GND</text>
+<text x="8.636" y="14.478" size="0.8128" layer="25" font="vector" ratio="10">bot-thoughts.com</text>
+<wire x1="4.572" y1="7.62" x2="4.572" y2="6.858" width="0.127" layer="21"/>
+<wire x1="4.572" y1="6.858" x2="4.572" y2="6.096" width="0.127" layer="21"/>
+<wire x1="4.572" y1="6.858" x2="5.08" y2="6.858" width="0.127" layer="21"/>
+<wire x1="5.08" y1="6.858" x2="6.35" y2="8.128" width="0.127" layer="21"/>
+<wire x1="6.35" y1="8.128" x2="8.89" y2="8.128" width="0.127" layer="21"/>
+<wire x1="10.668" y1="5.588" x2="16.002" y2="5.588" width="0.127" layer="21"/>
+<text x="10.16" y="4.064" size="0.8128" layer="25" font="vector" ratio="10" rot="R180" align="bottom-center">5V&gt;VDD</text>
+<wire x1="16.002" y1="6.604" x2="16.002" y2="5.588" width="0.127" layer="21"/>
+<wire x1="16.002" y1="5.588" x2="16.002" y2="4.318" width="0.127" layer="21"/>
 </plain>
 <attributes>
@@
 </autorouter>
 <elements>
-<element name="D1" library="ads4" package="SOD-323ORIG" value="" x="5.334" y="5.588" smashed="yes" rot="R270">
-<attribute name="VALUE" x="3.334" y="7.238" size="1.27" layer="27" font="vector" ratio="16" rot="R270"/>
+<element name="D1" library="ads4" package="SOD-323ORIG" value="" x="5.588" y="10.668" smashed="yes" rot="R90">
+<attribute name="VALUE" x="7.588" y="9.018" size="1.27" layer="27" font="vector" ratio="16" rot="R90"/>
 </element>
-<element name="J2" library="bt_avr" package="UPDI_1X3" value="UPDI COMPACT" x="12.7" y="8.128" smashed="yes" rot="MR180"/>
-<element name="U$1" library="bt" package="BTLOGOS" value="BTLOGO-LOGO-SM" x="6.604" y="13.716" rot="MR90"/>
+<element name="J2" library="bt_avr" package="UPDI_1X3" value="UPDI COMPACT" x="18.288" y="8.128" smashed="yes" rot="MR180"/>
+<element name="U$1" library="bt" package="BTLOGOS" value="BTLOGO-LOGO-SM" x="6.604" y="12.7"/>
 <element name="J3" library="bt_communication" package="6PIN_TARGET" value="6PIN SERIAL" x="1.778" y="8.128" smashed="yes"/>
+<element name="JMP1" library="bt" package="JUMPER-2W-PIN-0.1IN" value="PWR" x="10.16" y="8.128" smashed="yes" rot="R90"/>
 </elements>
 <signals>
-<signal name="N$2">
-<contactref element="J2" pad="3"/>
-<contactref element="D1" pad="A"/>
-<contactref element="J3" pad="5"/>
-<wire x1="1.778" y1="4.318" x2="5.314" y2="4.318" width="0.4064" layer="1"/>
-<wire x1="5.314" y1="4.318" x2="5.334" y2="4.338" width="0.4064" layer="1"/>
-<wire x1="5.334" y1="4.338" x2="6.37" y2="4.338" width="0.4064" layer="1"/>
-<wire x1="6.37" y1="4.338" x2="9.144" y2="7.112" width="0.4064" layer="1"/>
-<via x="9.144" y="7.112" extent="1-16" drill="0.3302"/>
-<wire x1="9.144" y1="7.112" x2="12.7" y2="10.668" width="0.4064" layer="16"/>
-</signal>
 <signal name="VCC">
 <contactref element="J2" pad="1"/>
-<contactref element="J3" pad="3"/>
-<wire x1="1.778" y1="9.398" x2="8.89" y2="9.398" width="0.4064" layer="1"/>
-<wire x1="8.89" y1="9.398" x2="12.7" y2="5.588" width="0.4064" layer="1"/>
-</signal>
-<signal name="N$1">
-<contactref element="D1" pad="C"/>
-<contactref element="J3" pad="4"/>
-<wire x1="1.778" y1="6.858" x2="5.314" y2="6.858" width="0.4064" layer="1"/>
-<wire x1="5.314" y1="6.858" x2="5.334" y2="6.838" width="0.4064" layer="1"/>
+<contactref element="JMP1" pad="1"/>
+<wire x1="18.288" y1="5.588" x2="10.16" y2="5.588" width="0.254" layer="1"/>
 </signal>
 <signal name="GND">
 <contactref element="J2" pad="2"/>
 <polygon width="0.4064" layer="16">
-<vertex x="11.938" y="0"/>
+<vertex x="0.635" y="16.256"/>
+<vertex x="19.431" y="16.256" curve="-90"/>
+<vertex x="20.066" y="15.621"/>
+<vertex x="20.066" y="0.635" curve="-90"/>
+<vertex x="19.431" y="0"/>
 <vertex x="0.635" y="0" curve="-90"/>
 <vertex x="0" y="0.635"/>
 <vertex x="0" y="15.621" curve="-90"/>
-<vertex x="0.635" y="16.256"/>
-<vertex x="11.938" y="16.256"/>
-<vertex x="14.478" y="13.716"/>
-<vertex x="14.478" y="2.54"/>
 </polygon>
-<contactref element="J3" pad="1"/>
+<contactref element="J3" pad="6"/>
+</signal>
+<signal name="N$1">
+<contactref element="J3" pad="3"/>
+<contactref element="D1" pad="C"/>
+<wire x1="5.588" y1="9.418" x2="1.778" y2="9.418" width="0.254" layer="1"/>
+<wire x1="1.778" y1="9.418" x2="1.778" y2="9.398" width="0.254" layer="1"/>
+</signal>
+<signal name="DATA">
+<contactref element="J3" pad="2"/>
+<contactref element="D1" pad="A"/>
+<contactref element="J2" pad="3"/>
+<wire x1="5.588" y1="11.918" x2="1.778" y2="11.918" width="0.254" layer="1"/>
+<wire x1="1.778" y1="11.918" x2="1.778" y2="11.938" width="0.254" layer="1"/>
+<wire x1="5.588" y1="11.918" x2="7.346" y2="11.918" width="0.254" layer="1"/>
+<wire x1="7.346" y1="11.918" x2="7.874" y2="12.446" width="0.254" layer="1"/>
+<wire x1="7.874" y1="12.446" x2="16.51" y2="12.446" width="0.254" layer="1"/>
+<wire x1="16.51" y1="12.446" x2="18.288" y2="10.668" width="0.254" layer="1"/>
+</signal>
+<signal name="N$2">
+<contactref element="J3" pad="4"/>
+<contactref element="JMP1" pad="2"/>
+<wire x1="1.778" y1="6.858" x2="5.08" y2="6.858" width="0.254" layer="1"/>
+<wire x1="5.08" y1="6.858" x2="6.35" y2="8.128" width="0.254" layer="1"/>
+<wire x1="6.35" y1="8.128" x2="10.16" y2="8.128" width="0.254" layer="1"/>
 </signal>
 </signals>
 </board>
 </drawing>
-<compatibility>
-<note version="6.3" minversion="6.2.2" severity="warning">
-Since Version 6.2.2 text objects can contain more than one line,
-which will not be processed correctly with this version.
-</note>
-</compatibility>
 </eagle>
