File: electronics/ftdi_adapter.brd (EAGLE design)
At the start: 20.1 x 16.3 mm, 5 parts, among them J2 UPDI COMPACT, J3 6PIN SERIAL

Commit message: Updated version #
Other:
- board text added: "R0.2"
- board text removed: "R0.1"
Changed lines of the file:
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@@
 <text x="11.684" y="1.016" size="1.016" layer="25" font="vector" ratio="10" align="bottom-center">UPDI Adapter</text>
 <text x="8.636" y="13.97" size="0.8128" layer="25" font="vector" ratio="10">cc-by-sa</text>
-<text x="19.558" y="1.27" size="0.8128" layer="25" font="vector" ratio="10" rot="R90">R0.1</text>
+<text x="19.558" y="1.27" size="0.8128" layer="25" font="vector" ratio="10" rot="R90">R0.2</text>
 <text x="17.018" y="10.922" size="0.8128" layer="25" font="vector" ratio="10" rot="R90" align="bottom-center">UPDI</text>
 <text x="17.018" y="5.588" size="0.8128" layer="25" font="vector" ratio="10" rot="R90" align="bottom-center">VDD</text>
