File: electronics/ftdi_adapter.sch (EAGLE design)
At the start: 5 parts, among them J2 UPDI COMPACT, J3 6PIN SERIAL

Commit message: Updated version #
Other:
- note added: "R0.2"
- note removed: "R0.1"
Changed lines of the file:
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@@
 <plain>
 <text x="154.94" y="17.78" size="3.81" layer="94">FTDI to UPDI Adapter</text>
-<text x="231.14" y="17.78" size="3.81" layer="94">R0.1</text>
+<text x="231.14" y="17.78" size="3.81" layer="94">R0.2</text>
 </plain>
 <instances>
